File: hardware/kicad/control_invernadero/control_invernadero.kicad_sch (KiCad schematic)
At the start: 33 parts, among them J1 Raspberry_Pi_2_3, J2 AC, J3 Ventilador2, J4 Ventilador 1, J5 Bomba de agua, Q2 IRLZ44N, Q3 IRLZ44N, Q4 IRLZ44N, U2 DS18B20, U3 DS18B20, U4 DS18B20, U5 DS18B20, U6 4N25, U7 MOC3021M, U8 Pico

Commit message: Esquematico actualizado
Parts:
- added J6: Sensor_humedad, symbol Connector:Screw_Terminal_01x03
Connections:
- net Earth: now also J6.GND
- net VCC Pi4: now also J6.VCC
- net at D2.2 (A), D3.1 (K), D3.2 (A)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: now also J2.Fase; no longer J2.2 (Pin_2)
- net at U8.31 (GPIO26_ADC0): now also J6.A0
- net at D4.2 (A), Puentedediodos.1 (K), R3.2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: now also J2.Neutro; no longer J2.1 (Pin_1)
Other:
- moved on the sheet: J2, J3, J4, J5, Lamp, Puentedediodos, Q2, Q3, Q4, R1, R10, R11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

Commit message: Se suben codigo PID y actualización del esquemático
Parts:
- R1: value 15K -> 68K
Changed lines of the file:
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@@
 			)
 		)
-		(property "Value" "15K"
+		(property "Value" "68K"
 			(at 250.19 78.7399 0)
 			(effects
